File: User Adapter/User Adapter.kicad_pcb (KiCad board)
At the start: 2 copper layers, 88.9 x 27.9 mm, 18 parts, among them J1 OHIS_8p8c_Shield, J2 Headphones, J3 Microphone, J4 PTT, J5 Dynamic Mic Bypass, J6 HP or CTIA, Q1 2N3904, SW1 SW_Push

Commit message: https://github.com/open-headset-interconnect-standard/ohis/issues/14 Streamed at https://youtube.com/live/3NY6S8Obg_s
Parts:
- added G***: LOGO, LOGO, B.Cu at (144.8, 84.5)
- added G1: Logo_OHIS, Libraries:Logo_OHIS_Medium, F.Cu at (171.4, 76.2)
- moved J6 2.53 mm to (133.3, 83.2)
- moved C1 1.27 mm to (156.2, 78.1)
- moved C2 1.27 mm to (157.5, 78.1)
- moved R1 1.27 mm to (160.7, 78.1)
- moved Q1 1.27 mm to (154.6, 70.5)
- moved R2 1.27 mm to (145.4, 67.9)
- moved R3 1.27 mm to (149.2, 67.9)
- moved J5 0.64 mm to (157.5, 81.9)
Routing:
- net HP:L: track 50.2 -> 83.4 mm, vias 0 -> 2
- net HP:R: track 54.4 -> 81.9 mm
- net Mic+: track 0.00 -> 27.0 mm
- net GND: track 0.00 -> 16.6 mm, vias 18 -> 56
- net Mic-: track 0.00 -> 13.9 mm, vias 63 -> 79
- net HP:G: track 0.00 -> 8.48 mm, vias 5 -> 41
- net PTT: track 93.1 -> 90.1 mm
- net Net-(J6-Pin_4): track 43.6 -> 46.2 mm
- net Net-(J5-Pin_1): track 5.70 -> 5.07 mm
- net Net-(J5-Pin_2): track 12.9 -> 12.3 mm
Other:
- board text added: "1nF"
- board text added: "1uF"
- board text added: "27k"
- board text added: "2N3904"
- board text added: "470"
- board text added: "75k"
- board text added: "CTIA"
- board text added: "Dynamic"
- board text added: "Electret"
- board text added: "Mic"
- board text added: "Mic Type"
- board text added: "OHIS Open Source User Adapter 2023 CC-BY OHIS Working Group"
- board text added: "PTT"
- board text added: "Phones"
- board text added: "https://github.com/open-headset-interconnect-standard/user-adapter"
