File: Top Board/Top Board.kicad_sch (KiCad schematic)
At the start: 5 parts

Commit message: Fixed silkscreen art, added trimpot. #1
Parts:
- G1: footprint Libraries:Logo_OHIS_Medium -> Libraries:Logo_OHIS_Large
Changed lines of the file:
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@@
       (effects (font (size 1.27 1.27)) hide)
     )
-    (property "Footprint" "Libraries:Logo_OHIS_Medium" (at 102.235 71.12 0)
+    (property "Footprint" "Libraries:Logo_OHIS_Large" (at 102.235 71.12 0)
       (effects (font (size 1.27 1.27)) hide)
     )
